File: isoSPI-M3Y-BMS-PCB.kicad_pcb (KiCad board)
At the start: 4 copper layers, 260 x 113 mm, 389 parts, among them J1 Screw_Terminal_01x04, J10 Screw_Terminal_01x04, J11 Screw_Terminal_01x03, J12 Screw_Terminal_01x08, J13 Conn_02x10_Odd_Even, J14 Screw_Terminal_01x04, J15 USB_C_Receptacle_USB2.0_16P, J16 Conn_01x03, J17 USB_C_Receptacle_USB2.0_16P, J18 USB_C_Receptacle_USB2.0_16P, J2 Conn_02x10_Odd_Even, J3 8P8C_LED_Shielded_x2, J5 OEM Shunt Connector, J6 349128020, J7 OEM HV Sense Connector, J8 OEM Connector, J9 Conn_01x03, Q1 CRSM034N06L2, Q2 CRSM034N06L2, Q3 CRSM034N06L2, Q5 CRSM034N06L2, SW1 TS-1187A-B-A-B, SW2 TS-1187A-B-A-B, SW3 TS-1187A-B-A-B, SW4 TS-1187A-B-A-B, U1 SN74LV1T08DBVR, U10 LTV-217-B-G, U11 RP2354B, U12 ADS1115, U13 ISO1050DUB, U15 SN74LV1T08DBVR, U16 BatMan, U17 TPS5430DDAR, U2 ISO1540, U20 LTV-217-B-G, U21 AMS1117-3.3, U22 F0505S-1WR3, U23 SN74LV1T08DBVR, U24 F0505S-1WR3, U25 SN74LV1T08DBVR, U26 SN74LV1T08DBVR, U27 RP2354B, U28 AM26LV32EIDR, U29 B0505S-3WR2, U3 INA228, U30 ISO1540, U32 SP3485EN-L/TR, U4 ISO1540, U6 F0505S-1WR3, U8 LTV-217-B-G, U9 LTV-217-B-G, Y1 ABM8-272-T3, Y2 ABM8-272-T3

Commit message: cleanup the pcb more
Parts:
- removed TH1, TH2, TH3, TH4, TH5, TH6: B59451C1130B070, BMS_Library:RV_Disc_D15.5mm_W7.5mm_P5.0mm
- moved R190 30.6 mm to (312.0, 285.7), turned to 180 degrees
- moved D23 30.5 mm to (307.7, 285.8), turned to 0 degrees
- moved D14 21.9 mm to (298.0, 313.6), turned to 180 degrees
- moved TP8 21.4 mm to (308.6, 279.1)
- moved C57 15.2 mm to (300.2, 303.5), turned to -90 degrees
- moved D50 15.0 mm to (256.5, 305.3)
- moved D51 15.0 mm to (256.5, 312.9)
- moved D18 15.0 mm to (256.5, 297.7)
- moved C2 12.8 mm to (271.6, 310.3), turned to 0 degrees
- moved R150 8.62 mm to (294.4, 304.6)
- moved D12 6.62 mm to (298.0, 318.6), turned to 180 degrees
- moved C132 6.31 mm to (307.8, 297.6), turned to 0 degrees
- moved R74 5.28 mm to (288.6, 309.5), turned to 180 degrees
- moved C1 5.05 mm to (283.6, 296.0)
- moved R148 4.88 mm to (291.1, 304.7), turned to 180 degrees
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Connections:
- J1 pad 1: /Logic_Input -> GND
- J1 pad 2: GND -> /Contactor_Input
- J1 pad 3: /Contactor_Input -> GND
- J1 pad 4: GND -> /Logic_Input
Routing:
- net +5V: track 31.8 -> 46.0 mm, vias 0 -> 1
- net /Logic_Input: track 4.71 -> 0.00 mm
- net IsoSPI-: track 25.2 -> 29.8 mm
- net IsoSPI+: track 24.9 -> 27.0 mm
