File: isoSPI-M3Y-BMS-PCB.kicad_pcb (KiCad board)
At the start: 4 copper layers, 260 x 113 mm, 398 parts, among them J1 Screw_Terminal_01x04, J10 Screw_Terminal_01x04, J11 Screw_Terminal_01x03, J12 Screw_Terminal_01x08, J13 Conn_02x10_Odd_Even, J14 Screw_Terminal_01x04, J15 USB_C_Receptacle_USB2.0_16P, J16 Conn_01x03, J17 USB_C_Receptacle_USB2.0_16P, J18 USB_C_Receptacle_USB2.0_16P, J2 Conn_02x10_Odd_Even, J3 8P8C_LED_Shielded_x2, J5 OEM Shunt Connector, J6 349128020, J7 OEM HV Sense Connector, J8 OEM Connector, J9 Conn_01x03, Q1 CRSM034N06L2, Q2 CRSM034N06L2, Q3 CRSM034N06L2, Q5 CRSM034N06L2, SW1 TS-1187A-B-A-B, SW2 TS-1187A-B-A-B, SW3 TS-1187A-B-A-B, SW4 TS-1187A-B-A-B, U1 SN74LV1T08DBVR, U10 LTV-217-B-G, U11 RP2354B, U12 ADS1115, U13 ISO1050DUB, U15 SN74LV1T08DBVR, U16 BatMan, U17 TPS5430DDAR, U2 ISO1540, U20 LTV-217-B-G, U21 AMS1117-3.3, U22 F0505S-1WR3, U23 SN74LV1T08DBVR, U24 F0505S-1WR3, U25 SN74LV1T08DBVR, U26 SN74LV1T08DBVR, U27 RP2354B, U28 AM26LV32EIDR, U29 B0505S-3WR2, U3 INA228, U30 ISO1540, U32 SP3485EN-L/TR, U4 ISO1540, U6 F0505S-1WR3, U8 LTV-217-B-G, U9 LTV-217-B-G, Y1 ABM8-272-T3, Y2 ABM8-272-T3

Commit message: more updates
Parts:
- added TP15: TestPoint_2Pole, BMS_Library:TestPoint_2Pads_Pitch2.54mm_Pad1.5_Drill1.0mm, F.Cu at (428.6, 249.0)
- added TP16: TestPoint_2Pole, BMS_Library:TestPoint_2Pads_Pitch2.54mm_Pad1.5_Drill1.0mm, F.Cu at (428.6, 244.9)
- added TP19: TestPoint_2Pole, BMS_Library:TestPoint_2Pads_Pitch2.54mm_Pad1.5_Drill1.0mm, F.Cu at (474.5, 258.6)
- TP1, TP17, TP18, TP2, TP3, TP4, TP5, TP6, TP7, TP8, TP9: footprint bms:TestPoint_2Pads_Pitch2.54mm_Drill0.9mm -> BMS_Library:TestPoint_2Pads_Pitch2.54mm_Pad1.5_Drill1.0mm
- moved R67 13.6 mm to (420.6, 245.1)
- moved R66 13.6 mm to (420.7, 248.3)
- moved R141 3.67 mm to (472.2, 262.1), turned to -90 degrees
- moved TP5 3.35 mm to (445.9, 255.7)
- moved C24 2.29 mm to (469.6, 262.6), turned to 0 degrees
- moved D38 1.68 mm to (475.2, 262.6)
- moved D40 1.09 mm to (475.3, 254.6)
- moved R142 0.99 mm to (472.5, 255.3), turned to 90 degrees

Commit message: connect remaining gpio
Connections:
- U27 pad 14: /GPIO15 -> FC-Neg
- U27 pad 16: /GPIO16 -> Neg
- U27 pad 17: /GPIO17 -> Pos
- U27 pad 18: /GPIO18 -> FC-Pos
- U27 pad 19: /GPIO19 -> CAN Rx
- U27 pad 20: /GPIO20 -> CAN Tx
- U27 pad 21: /GPIO21 -> I2C SCL Vsense
- U27 pad 22: /GPIO22 -> I2C SDA Vsense
- U27 pad 23: /GPIO23 -> I2C SCL Shunt
- U27 pad 25: /GPIO24 -> I2C SDA Shunt

Commit message: progress...
Parts:
- added C76: 100nF, Capacitor_SMD:C_0603_1608Metric, F.Cu at (416.5, 305.8)
- JP9: value SolderJumper_3_Bridged12 -> SolderJumper_2_Bridged; footprint Jumper:SolderJumper-3_P1.3mm_Bridged12_RoundedPad1.0x1.5mm_NumberLabels -> Jumper:SolderJumper-2_P1.3mm_Bridged_RoundedPad1.0x1.5mm
- moved J16 20.2 mm to (430.8, 243.8), turned to 90 degrees
- moved J9 20.1 mm to (355.6, 243.2), turned to 90 degrees
- moved R100 12.0 mm to (350.3, 285.2), turned to 150 degrees
- moved R101 11.6 mm to (382.4, 285.7), turned to -150 degrees
- moved R63 10.5 mm to (396.2, 240.9), turned to 180 degrees
- moved R104 10.4 mm to (348.6, 288.0), turned to -30 degrees
- moved R105 9.97 mm to (384.0, 288.6), turned to 30 degrees
- moved TP16 9.06 mm to (435.3, 250.9), turned to 90 degrees
- moved TP15 8.94 mm to (434.1, 256.1)
- moved R108 8.92 mm to (347.0, 290.9), turned to 150 degrees
- moved R64 8.90 mm to (396.3, 243.5), turned to 180 degrees
- moved R109 8.41 mm to (385.6, 291.4), turned to -150 degrees
- moved R115 7.48 mm to (345.4, 293.7), turned to -30 degrees
- moved R116 6.93 mm to (387.2, 294.2), turned to 30 degrees
- moved R99 6.38 mm to (454.5, 321.2), turned to 0 degrees
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Connections:
- net Shunt NTC - renamed GND Shunt NTC -
- C85 pad 2: Net-(JP9-A) -> Net-(JP9-B)
- J15 pad A6: /Serial API RX -> /Serial API TX
- J15 pad A7: /Serial API TX -> /Serial API RX
- J15 pad B6: /Serial API RX -> /Serial API TX
- J15 pad B7: /Serial API TX -> /Serial API RX
- J2 pad 10: /GPIO8 -> /GPIO7
- J2 pad 12: /GPIO9 -> /GPIO8
- J2 pad 14: /GPIO10 -> /GPIO9
- J2 pad 16: /GPIO11 -> /GPIO10
- J2 pad 18: /GPIO12 -> /GPIO11
- J2 pad 2: /GPIO4 -> /GPIO3
- J2 pad 20: /GPIO13 -> /GPIO12
- J2 pad 4: /GPIO5 -> /GPIO4
- J2 pad 6: /GPIO6 -> /GPIO5
- J2 pad 8: /GPIO7 -> /GPIO6
- JP9 pad 2: Net-(JP9-C) -> Net-(JP9-B)
- R63 pad 1: MUC1-MCU2 TX-RX -> SUP-MAIN TX/RX
- R63 pad 2: /GPIO1 -> /MCU2_GPIO1
- R64 pad 1: MUC2-MCU1 TX-RX -> MAIN-SUP TX/RX
- R64 pad 2: /GPIO2 -> /MCU2_GPIO2
- TP9 pad 1: MUC2-MCU1 TX-RX -> SUP-MAIN TX/RX
- TP9 pad 2: MUC1-MCU2 TX-RX -> MAIN-SUP TX/RX
- TR10 pad 2: Net-(JP9-C) -> Net-(JP9-A)
- U11 pad 36: /MCU2_GPIO28 -> IsoSPI RX H
- U11 pad 37: /MCU2_GPIO29 -> IsoSPI RX L
- U11 pad 38: /MCU2_GPIO30 -> IsoSPI RX AND
- U11 pad 39: /MCU2_GPIO31 -> IsoSPI RX Debug
- U11 pad 40: /MCU2_GPIO32 -> Snooper Debug
- U11 pad 78: MUC2-MCU1 TX-RX -> /MCU2_GPIO1
- U11 pad 79: MUC1-MCU2 TX-RX -> /MCU2_GPIO2
- U27 pad 12: /GPIO13 -> Extra Output 1
- U27 pad 13: /GPIO14 -> Extra Output 2
- U27 pad 78: /GPIO1 -> MAIN-SUP TX/RX
- U27 pad 79: /GPIO2 -> SUP-MAIN TX/RX
Routing:
- net C_En: track 0.00 -> 125.3 mm
- net /CAN L: track 0.00 -> 54.2 mm, vias 0 -> 8
- net Net-(C40-Pad1): track 0.00 -> 51.8 mm, vias 0 -> 1
- net /QSPI2_SS: track 0.00 -> 47.7 mm, vias 0 -> 2
- net /CAN H: track 0.00 -> 44.0 mm, vias 0 -> 2
- net Net-(J3-Pad15): track 0.00 -> 43.7 mm, vias 0 -> 1
- net Net-(C26-Pad1): track 0.00 -> 43.6 mm
- net /CAN 5V: track 0.00 -> 43.3 mm
- net /RUN_2: track 0.00 -> 39.9 mm
- net GND: track 39.0 -> 77.7 mm, vias 53 -> 59
- net Shunt_5V: track 0.00 -> 34.4 mm
- net Net-(J3-Pad17): track 0.00 -> 32.7 mm
- net Net-(J3-Pad16): track 0.00 -> 31.7 mm, vias 0 -> 1
- net Net-(J3-Pad18): track 0.00 -> 30.0 mm
- net /Serial API TX: track 0.00 -> 27.2 mm
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- added copper zone on B.Cu, net +3.3V
- added copper zone on In2.Cu, net GND
- added copper zone on In2.Cu, net GND CAN
- added copper zone on In2.Cu, net GND Shunt NTC -
- added copper zone on In2.Cu, net GND_RS
- added copper zone on In2.Cu, net GND_VSens
- removed copper zone on In2.Cu, net +3.3V
- removed copper zone on In2.Cu, net +5V
Other:
- board text added: "L"
- board text added: "Main RP2354B"
- board text added: "Supervisor RP2354B"
- board text removed: "Main"
- board text removed: "Supervisor"
