File: isoSPI-M3Y-BMS-PCB.kicad_sch (KiCad schematic)
At the start: 428 parts, among them J1 Screw_Terminal_01x04, J10 Screw_Terminal_01x04, J11 Screw_Terminal_01x03, J12 Screw_Terminal_01x08, J13 Conn_02x10_Odd_Even, J14 Screw_Terminal_01x04, J15 USB_C_Receptacle_USB2.0_16P, J16 Conn_01x03, J17 USB_C_Receptacle_USB2.0_16P, J18 USB_C_Receptacle_USB2.0_16P, J2 Conn_02x10_Odd_Even, J3 8P8C_LED_Shielded_x2, J5 OEM Shunt Connector, J6 349128020, J7 OEM HV Sense Connector, J8 OEM Connector, J9 Conn_01x03, K1 FC Positive, K10 FC Positive, K11 FC Negative, K12 Link Negative, K13 Inverter, K14 Link Positive, K15 Link Negative, K16 FC Positive, K17 FC Negative, K18 Inverter, K2 FC Negative, K3 Link Negative, K4 Link Positive, K5 Link Positive, K6 FC Positive, K7 FC Negative, K8 Link Negative, K9 Link Positive, Q1 CRSM034N06L2, Q2 CRSM034N06L2, Q3 CRSM034N06L2, Q5 CRSM034N06L2, SW1 TS-1187A-B-A-B, SW2 TS-1187A-B-A-B, SW3 TS-1187A-B-A-B, SW4 TS-1187A-B-A-B, U1 SN74LV1T08DBVR, U10 LTV-217-B-G, U11 RP2354B, U12 ADS1115, U13 ISO1050DUB, U15 SN74LV1T08DBVR, U16 BatMan, U17 TPS5430DDAR, U2 ISO1540, U20 LTV-217-B-G, U21 AMS1117-3.3, U22 F0505S-1WR3, U23 SN74LV1T08DBVR, U24 F0505S-1WR3, U25 SN74LV1T08DBVR, U26 SN74LV1T08DBVR, U27 RP2354B, U28 AM26LV32EIDR, U29 B0505S-3WR2, U3 INA228, U30 ISO1540, U32 SP3485EN-L/TR, U4 ISO1540, U6 F0505S-1WR3, U8 LTV-217-B-G, U9 LTV-217-B-G, Y1 ABM8-272-T3, Y2 ABM8-272-T3

Commit message: update gitignore
Parts:
- removed F3, F4: Pyro Fuse, symbol Device:Fuse
- removed K1, K6: FC Positive, symbol Relay:Fujitsu_FTR-LYAA005x
- removed K2, K7: FC Negative, symbol Relay:Fujitsu_FTR-LYAA005x
- removed K3, K8: Link Negative, symbol Relay:Fujitsu_FTR-LYAA005x
- removed K4, K5: Link Positive, symbol Relay:Fujitsu_FTR-LYAA005x
- removed R163, R166: R_Shunt, symbol Device:R_Shunt
- removed R164, R165: 27R, symbol Device:R_US
Other:
- moved on the sheet: BT1, BT3, BT4, BT5, BT6, BT7, BT8, BT9, F1, F11, F8, F9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

Commit message: cleanup the pcb more
Connections:
- net Contactor_Input: now also J1.2 (Pin_2); no longer J1.3 (Pin_3)
- net GND: now also J1.1 (Pin_1), J1.3 (Pin_3); no longer J1.2 (Pin_2), J1.4 (Pin_4)
- net Logic_Input: now also J1.4 (Pin_4); no longer J1.1 (Pin_1)
Other:
- note added: "ENA enabled while NC"
- note removed: "enabled while NC"
- moved on the sheet: BT1, BT3, BT4, BT5, C57, F8, F9, J1, K10, K11, K12, K13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
