File: isoSPI-M3Y-BMS-PCB.kicad_sch (KiCad schematic)
At the start: 456 parts, among them J1 Screw_Terminal_01x04, J10 Screw_Terminal_01x04, J11 3.81P Screw Terminal, J12 3.81P Screw Terminal, J13 Conn_02x10_Odd_Even, J14 Screw_Terminal_01x04, J15 USB_C_Receptacle_USB2.0_16P, J16 Conn_01x03, J17 USB_C_Receptacle_USB2.0_16P, J18 USB_C_Receptacle_USB2.0_16P, J19 Conn_01x04, J2 Conn_02x10_Odd_Even, J20 Screw_Terminal_01x04, J3 8P8C_LED_Shielded_x2, J4 Conn_01x04, J5 OEM Shunt Connector, J6 349128020, J7 OEM HV Sense Connector, J8 OEM Connector, J9 Conn_01x03, K10 FC Positive, K11 FC Negative, K12 Link Negative, K13 Inverter, K14 Link Positive, K15 Link Negative, K16 FC Positive, K17 FC Negative, K18 Inverter, K9 Link Positive, Q1 CRSM034N06L2, Q2 CRSM034N06L2, Q3 CRSM034N06L2, Q5 CRSM034N06L2, SW1 TS-1187A-B-A-B, SW2 TS-1187A-B-A-B, SW3 TS-1187A-B-A-B, SW4 TS-1187A-B-A-B, U1 SN74LV1T08DBVR, U10 LTV-217-B-G, U11 RP2354B, U12 ADS1115, U13 ISO1050DUB, U15 SN74LV1T08DBVR, U16 BatMan, U17 TPS5430DDAR, U2 ISO1540, U20 LTV-217-B-G, U21 AMS1117-3.3, U22 F0505S-1WR3, U23 SN74LV1T08DBVR, U24 F0505S-1WR3, U25 SN74LV1T08DBVR, U26 SN74LV1T08DBVR, U27 RP2354B, U28 AM26LV32EIDR, U29 B0505S-3WR2, U3 INA228, U30 ISO1540, U32 SP3485EN-L/TR, U4 ISO1540, U5 LTV-217-B-G, U6 F0505S-1WR3, U7 LTV-217-B-G, U8 LTV-217-B-G, U9 LTV-217-B-G, Y1 ABM8-272-T3, Y2 ABM8-272-T3

Commit message: lots more
Parts:
- removed J19, J4: Conn_01x04, Connector_PinHeader_2.54mm:PinHeader_1x04_P2.54mm_Vertical, symbol Connector_Generic:Conn_01x04
- added H10, H11, H14, H15, H16, H9: Mouse Bites 2mm, BMS_Library:mouse-bite-2mm-slot-min, symbol Mechanical:MountingHole
- added TP31, TP32, TP33, TP34, TP35, TP36, TP37, TP38: TP, BMS_Library:TestPoint_THTPad_D1.5mm_Drill1.0mm, symbol Connector:TestPoint_Small
- C112, C34, C69: Field5 C46550429 -> (none); JLCPCB Part # (none) -> C46550429
- H1, H12, H13, H2, H3, H4, H5, H7, J1, J10, J11, J12, J13, J14, J2, J20, U16: now not fitted
- J15, J17, J18: JLCPCB Part # (none) -> C2765186
- J5: JLCPCB Part # (none) -> C17284895; MFR.Part # (none) -> ZE05H-8DP-2H; now not fitted
- J6: value 349128020 -> OEM Connector; Field6 OEM Connector -> (none); MFR.Part # (none) -> 349128020
- J7: JLCPCB Part # (none) -> C573648; MFR Part # (none) -> 173864-1; now not fitted
- J8: Mfr. # (none) -> S44B-RAD1AK; now not fitted
- L6, L7: value 3.3u -> 3.3uh; Field6JJLCPCB Part # C42411119 -> (none); JLCPCB Part # (none) -> C42411119
- R141: JLCPCB Part # DNP -> (none); now not fitted
- U10, U20, U22, U24, U29, U5, U6, U7, U8, U9: FT Rotation Offset (none) -> 90
Connections:
- net Emergency Stop: now also J13.18 (Pin_18); no longer J13.16 (Pin_16)
- net GND: now also TP31.1, TP35.1
- net MCU2_GPIO10: now also J13.16 (Pin_16); no longer J13.14 (Pin_14)
- net MCU2_GPIO12: now also J13.20 (Pin_20); no longer J13.18 (Pin_18)
- net MCU2_GPIO13: no longer J13.20 (Pin_20)
- net MCU2_GPIO3: now also J13.2 (Pin_2)
- net MCU2_GPIO4: now also J13.4 (Pin_4); no longer J13.2 (Pin_2)
- net MCU2_GPIO5: now also J13.6 (Pin_6); no longer J13.4 (Pin_4)
- net MCU2_GPIO6: now also J13.8 (Pin_8); no longer J13.6 (Pin_6)
- net MCU2_GPIO7: now also J13.10 (Pin_10); no longer J13.8 (Pin_8)
- net MCU2_GPIO8: now also J13.12 (Pin_12); no longer J13.10 (Pin_10)
- net MCU2_GPIO9: now also J13.14 (Pin_14); no longer J13.12 (Pin_12)
- net USB2_D+: now also TP36.1
- net USB2_D-: now also TP37.1
- net USB_D+: now also TP32.1
- net USB_D-: now also TP34.1
- net at D30.2 (A), J17.A4 (VBUS), J17.A9 (VBUS)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: now also TP38.1
- net at D53.2 (A), J18.A4 (VBUS), J18.A9 (VBUS)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: now also TP33.1
Other:
- moved on the sheet: J6, TP30
