File: CellKeeper.kicad_pcb (KiCad board)
At the start: 4 copper layers, 306 x 113 mm, 503 parts, among them J1 Screw_Terminal_01x04, J10 3.81P Screw Terminal, J11 USB_C_Receptacle_USB2.0_16P, J12 Conn_02x10_Odd_Even, J14 OEM Shunt Connector, J15 Screw_Terminal_01x04, J16 Conn_01x03, J17 OEM HV Sense Connector, J18 7.62mm Pitch Screw Terminal, J19 USB_C_Receptacle_USB2.0_16P, J2 Screw_Terminal_01x01, J20 OEM Connector, J21 3.81P Screw Terminal, J22 Conn_02x10_Odd_Even, J23 OEM Connector, J24 3.81P Screw Terminal, J3 Screw_Terminal_01x04, J4 8P8C_LED_Shielded_x2, J5 8P8C_LED_Shielded_x2, J6 OEM Connector, J7 Screw_Terminal_01x04, J8 Conn_01x03, J9 USB_C_Receptacle_USB2.0_16P, Q1 BSC0805LS, Q2 BSC0805LS, Q3 BSC0805LS, Q4 BSC0805LS, SW1 TS-1187A-B-A-B, SW2 TS-1187A-B-A-B, SW3 TS-1187A-B-A-B, SW4 TS-1187A-B-A-B, U1 UCC27524DR, U10 ISO1050DUB, U11 UCC27524DR, U12 LTV-217-B-G, U13 LTV-217-B-G, U14 RP2354B, U15 F0505S-1WR3, U16 ISO1540, U17 INA228, U18 ADS1115, U19 ADS1115, U2 AMS1117-3.3, U20 RP2354B, U21 SP3485EN-L/TR, U22 AM26LV32EIDR, U23 SP3485EN-L/TR, U24 AM26LV32EIDR, U3 TPS5430DDAR, U4 F0505S-1WR3, U5 ISO1050DUB, U6 LTV-217-B-G, U7 LTV-217-B-G, U8 LTV-217-B-G, U9 LTV-217-B-G, Y1 ABM8-272-T3, Y2 ABM8-272-T3

Commit message: start on rev1.1
Parts:
- removed R17, R6: 24k, CellKeeper_Local:Resistor_SMD__R_0603_1608Metric
- removed kibuzzard-6A48285D: G***, kibuzzard-6A48285D
- added JP37: 0r, CellKeeper_Local:BMS_Library__J_0603_jumper, F.Cu at (274.6, 126.1)
- added R151: 100k, CellKeeper_Local:Resistor_SMD__R_0603_1608Metric, F.Cu at (95.4, 134.4)
- added R152: 100k, CellKeeper_Local:Resistor_SMD__R_0603_1608Metric, F.Cu at (90.1, 134.3)
- added kibuzzard-6A6094FF: G***, kibuzzard-6A6094FF, F.Cu at (93.6, 44.6)
- J4, J5: footprint CellKeeper_Local:Connector_RJ__RJ45_Amphenol_RJHSE538X-02 -> CellKeeper_Local:Connector_RJ__RJ45_HCTL_HC-RJ45-5JA-2-2-Y
Routing:
- net Net-(TH3-Pad2): track 22.2 -> 44.4 mm
- net Net-(TH2-Pad2): track 22.3 -> 44.5 mm
- net Net-(TH1-Pad2): track 22.3 -> 44.5 mm
- net Net-(C19-Pad2): track 19.9 -> 22.1 mm
- net Net-(J4-Pad18): track 35.3 -> 36.6 mm
- net GND CAN: track 31.0 -> 31.8 mm, vias 8 -> 9
- added copper zone on B.Cu, net /FC Neg
- added copper zone on F.Cu, net /FC Neg
- added copper zone on In1.Cu, net /FC Neg
- added copper zone on In2.Cu, net /FC Neg
- added copper zone on B.Cu, net Drive Unit Neg
- added copper zone on F.Cu, net Drive Unit Neg
- added copper zone on In1.Cu, net Drive Unit Neg
- added copper zone on In2.Cu, net Drive Unit Neg
Other:
- board text added: "E-Stop"
- board text added: "Experimental PCS Jumpers"
- board text added: "FC AUX"
- board text added: "FC-P-AUX FC-N-AUX GND GND"
- board text added: "REV 1.1"
- board text removed: "Aux contacts - optional"
- board text removed: "FC-P-SW FC-N-SW GND GND"
- board text removed: "REV 1"
- board text removed: "optional"
