File: CellKeeper.kicad_pcb (KiCad board)
At the start: 4 copper layers, 306 x 113 mm, 504 parts, among them J1 Screw_Terminal_01x04, J10 3.81P Screw Terminal, J11 USB_C_Receptacle_USB2.0_16P, J12 Conn_02x10_Odd_Even, J14 OEM Shunt Connector, J15 Screw_Terminal_01x04, J16 Conn_01x03, J17 OEM HV Sense Connector, J18 7.62mm Pitch Screw Terminal, J19 USB_C_Receptacle_USB2.0_16P, J2 Screw_Terminal_01x01, J20 OEM Connector, J21 3.81P Screw Terminal, J22 Conn_02x10_Odd_Even, J23 OEM Connector, J24 3.81P Screw Terminal, J3 Screw_Terminal_01x04, J4 8P8C_LED_Shielded_x2, J5 8P8C_LED_Shielded_x2, J6 OEM Connector, J7 Screw_Terminal_01x04, J8 Conn_01x03, J9 USB_C_Receptacle_USB2.0_16P, Q1 BSC0805LS, Q2 BSC0805LS, Q3 BSC0805LS, Q4 BSC0805LS, SW1 TS-1187A-B-A-B, SW2 TS-1187A-B-A-B, SW3 TS-1187A-B-A-B, SW4 TS-1187A-B-A-B, U1 UCC27524DR, U10 ISO1050DUB, U11 UCC27524DR, U12 LTV-217-B-G, U13 LTV-217-B-G, U14 RP2354B, U15 F0505S-1WR3, U16 ISO1540, U17 INA228, U18 ADS1115, U19 ADS1115, U2 AMS1117-3.3, U20 RP2354B, U21 SP3485EN-L/TR, U22 AM26LV32EIDR, U23 SP3485EN-L/TR, U24 AM26LV32EIDR, U3 TPS5430DDAR, U4 F0505S-1WR3, U5 ISO1050DUB, U6 LTV-217-B-G, U7 LTV-217-B-G, U8 LTV-217-B-G, U9 LTV-217-B-G, Y1 ABM8-272-T3, Y2 ABM8-272-T3

Commit message: added 3v3 regulator to the INA228 isolated zone
Parts:
- removed R78: 24k, CellKeeper_Local:Resistor_SMD__R_0603_1608Metric
- removed U2: AMS1117-3.3, CellKeeper_Local:Package_TO_SOT_SMD__SOT-223-3_TabPin2
- added R17: 10k, CellKeeper_Local:Resistor_SMD__R_0603_1608Metric, F.Cu at (228.7, 121.1)
- added TP49: TP, CellKeeper_Local:BMS_Library__TestPoint_THTPad_D1.5mm_Drill1.0mm, F.Cu at (238.2, 131.7)
- added U25: TLV1117LV33DCYR, CellKeeper_Local:Package_TO_SOT_SMD__SOT-223-3_TabPin2, F.Cu at (140.2, 72.3)
- added U26: TLV1117LV33DCYR, CellKeeper_Local:Package_TO_SOT_SMD__SOT-223-3_TabPin2, F.Cu at (241.3, 136.5)
- moved TP18 18.4 mm to (244.6, 131.6)
- moved R73 8.13 mm to (242.1, 130.7), turned to 180 degrees
- moved FB3 3.64 mm to (244.6, 129.0), turned to -90 degrees
- moved C55 2.11 mm to (241.9, 128.8)
- moved R22 1.22 mm to (283.6, 124.1)
- moved R43 0.98 mm to (286.7, 124.1)
- moved JP37 0.90 mm to (273.7, 126.1)
- moved TH4 0.12 mm to (321.9, 92.8)
- moved TH5 0.12 mm to (321.9, 102.3)
- moved C54 0.06 mm to (236.4, 120.6)
Connections:
- C54 pad 2: Shunt_5V -> Shunt_3V3
- C57 pad 2: Shunt_5V -> Shunt_3V3
- C60 pad 2: Shunt_5V -> Shunt_3V3
- R69 pad 1: Shunt_5V -> Shunt_3V3
- R72 pad 1: Shunt_5V -> Shunt_3V3
- R84 pad 2: Shunt_5V -> Shunt_3V3
- U16 pad 8: Shunt_5V -> Shunt_3V3
- U17 pad 6: Shunt_5V -> Shunt_3V3
Routing:
- net Shunt_3V3: track 0.00 -> 47.4 mm
- net Net-(TH2-Pad2): track 44.5 -> 0.00 mm
- net Net-(TH1-Pad2): track 44.5 -> 0.00 mm
- net Net-(TH3-Pad2): track 44.4 -> 0.00 mm
- net Shunt_5V: track 48.0 -> 6.84 mm
- net GND Shunt NTC -: track 75.5 -> 82.5 mm, vias 6 -> 8
- net Net-(U15-+Vout): track 8.64 -> 5.31 mm
- net Net-(C19-Pad1): track 61.1 -> 63.3 mm
- net Shunt Sense -: track 29.1 -> 31.3 mm
- net Net-(C19-Pad2): track 22.1 -> 23.4 mm
- net /CAN 5V: track 58.9 -> 59.9 mm
- net Net-(J4-Pad22): track 16.3 -> 15.3 mm
- added copper zone on B.Cu, net Net-(TH1-Pad2)
- added copper zone on F.Cu, net Net-(TH1-Pad2)
- added copper zone on In1.Cu, net Net-(TH1-Pad2)
- added copper zone on In2.Cu, net Net-(TH1-Pad2)
- added copper zone on B.Cu, net Net-(TH2-Pad2)
- added copper zone on F.Cu, net Net-(TH2-Pad2)
- added copper zone on In1.Cu, net Net-(TH2-Pad2)
- added copper zone on In2.Cu, net Net-(TH2-Pad2)
- added copper zone on B.Cu, net Net-(TH3-Pad2)
- added copper zone on F.Cu, net Net-(TH3-Pad2)
- added copper zone on In1.Cu, net Net-(TH3-Pad2)
- added copper zone on In2.Cu, net Net-(TH3-Pad2)
- added copper zone on F.Cu, net Shunt_3V3
Other:
- board text added: "E-STOP"
- board text added: "H3, H4 fit mount in penthouse"
- board text added: "IMPORTANT connect chassis GND first"
- board text removed: "E-Stop"
- board text removed: "IMPORTANT Always Connect First"
