File: CellKeeper.kicad_sch (KiCad schematic)
At the start: 525 parts, among them J1 Screw_Terminal_01x04, J10 3.81P Screw Terminal, J11 USB_C_Receptacle_USB2.0_16P, J12 Conn_02x10_Odd_Even, J13 USB_C_Receptacle_USB2.0_16P, J14 OEM Shunt Connector, J15 Screw_Terminal_01x04, J16 Conn_01x03, J17 OEM HV Sense Connector, J18 7.62mm Pitch Screw Terminal, J19 USB_C_Receptacle_USB2.0_16P, J2 Screw_Terminal_01x01, J20 OEM Connector, J21 3.81P Screw Terminal, J22 Conn_02x10_Odd_Even, J23 OEM Connector, J24 3.81P Screw Terminal, J3 Screw_Terminal_01x04, J4 8P8C_LED_Shielded_x2, J5 8P8C_LED_Shielded_x2, J6 OEM Connector, J7 Screw_Terminal_01x04, J8 Conn_01x03, J9 USB_C_Receptacle_USB2.0_16P, K1 Link Positive, K10 Inverter, K2 Link Negative, K3 FC Positive, K4 FC Negative, K5 Inverter, K6 Link Positive, K7 Link Negative, K8 FC Negative, K9 FC Positive, Q1 BSC0805LS, Q2 BSC0805LS, Q3 BSC0805LS, Q4 BSC0805LS, SW1 TS-1187A-B-A-B, SW2 TS-1187A-B-A-B, SW3 TS-1187A-B-A-B, SW4 TS-1187A-B-A-B, U1 UCC27524DR, U10 ISO1050DUB, U11 UCC27524DR, U12 LTV-217-B-G, U13 LTV-217-B-G, U14 RP2354B, U15 F0505S-1WR3, U16 ISO1540, U17 INA228, U18 ADS1115, U19 ADS1115, U2 AMS1117-3.3, U20 RP2354B, U21 SP3485EN-L/TR, U22 AM26LV32EIDR, U23 SP3485EN-L/TR, U24 AM26LV32EIDR, U3 TPS5430DDAR, U4 F0505S-1WR3, U5 ISO1050DUB, U6 LTV-217-B-G, U7 LTV-217-B-G, U8 LTV-217-B-G, U9 LTV-217-B-G, Y1 ABM8-272-T3, Y2 ABM8-272-T3

Commit message: start on rev1.1
Parts:
- removed R17, R6: 24k, CellKeeper_Local:Resistor_SMD__R_0603_1608Metric, symbol CellKeeper_Local:Device__R_Small
- added JP37: 0r, CellKeeper_Local:BMS_Library__J_0603_jumper, symbol CellKeeper_Local:BMS_Library__Jumper_Resistor
- added R151, R152: 100k, CellKeeper_Local:Resistor_SMD__R_0603_1608Metric, symbol CellKeeper_Local:Device__R_Small
Connections:
- net GND CAN: now also JP37.2
- net Logic_Input: now also R151.2
- net V_{Contactor}: now also R152.2
- net at D13.2 (A): now also R151.1
- net at D22.2 (A): now also R152.1
- net at C19.1, J4.20, J4.21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: now also JP37.1
Other:
- note added: "E-Stop Disable"
- moved on the sheet: R22

Commit message: added 3v3 regulator to the INA228 isolated zone
Parts:
- removed R78: 24k, CellKeeper_Local:Resistor_SMD__R_0603_1608Metric, symbol CellKeeper_Local:Device__R_Small
- removed U2: AMS1117-3.3, CellKeeper_Local:Package_TO_SOT_SMD__SOT-223-3_TabPin2, symbol CellKeeper_Local:Regulator_Linear__AMS1117-3.3
- added R17: 10k, CellKeeper_Local:Resistor_SMD__R_0603_1608Metric, symbol CellKeeper_Local:Device__R_Small
- added TP49: TP, CellKeeper_Local:BMS_Library__TestPoint_THTPad_D1.5mm_Drill1.0mm, symbol CellKeeper_Local:Connector__TestPoint_Small
- added U25, U26: TLV1117LV33DCYR, CellKeeper_Local:Package_TO_SOT_SMD__SOT-223-3_TabPin2, symbol CellKeeper_Local:Regulator_Linear__AMS1117-3.3
Connections:
- net +3.3V: now also U25.2 (VO)
- net +LDO_IN: now also U25.3 (VI)
- net GND: now also U25.1 (GND)
- net GND_Shunt: now also U26.1 (GND)
- net Shunt_5V: now also U26.3 (VI); no longer C54.2, C57.2, C60.2, R69.1, R72.1, R84.2, U16.8 (VCC2), U17.6 (VS)
- net at D45.2 (A): now also R17.2
- new net Shunt_3V3: C54.2, C57.2, C60.2, R17.1, R69.1, R72.1, R84.2, TP49.1, U16.8 (VCC2), U17.6 (VS), U26.2 (VO)
Other:
- note added: "Specified DC-DC is the smaller package 3kV footprint will fit the 3kV or 6kV version H0505S-1WR2 = 6kV F0505S-1WR3 = 3kV - DC-DC output is 5.55v nominal with 5.2V input"
- note removed: "Specified DC-DC is the smaller package 3kV footprint will fit the 3kV or 6kV version H0505S-1WR2 = 6kV F0505S-1WR3 = 3kV"
- moved on the sheet: C22, C57, C60, C62, C64, D17, D45, J14, J15, R15, R20, R21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

Commit message: Work
Parts:
- removed C57: 1uF, CellKeeper_Local:Capacitor_SMD__C_0603_1608Metric, symbol CellKeeper_Local:Device__C_Small
- added C116: 10uF, CellKeeper_Local:Capacitor_SMD__C_0805_2012Metric, symbol CellKeeper_Local:Device__C_Small
Connections:
- net GND_Shunt: now also C116.1
- net Shunt_3V3: now also C116.2
Changed lines of the file:
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@@
 	)
 	(symbol
+		(lib_id "CellKeeper_Local:Device__C_Small")
+		(at 391.16 299.72 180)
+		(unit 1)
+		(body_style 1)
+		(exclude_from_sim no)
+		(in_bom yes)
+		(on_board yes)
+		(in_pos_files yes)
+		(dnp no)
+		(property "Reference" "C116"
+			(at 393.192 298.704 0)
+			(show_name no)
+			(do_not_autoplace no)
+			(effects
+				(font
+					(size 1.27 1.27)
+				)
+				(justify right)
+			)
+		)
+		(property "Value" "10uF"
+			(at 393.192 300.482 0)
+			(show_name no)
+			(do_not_autoplace no)
+			(effects
+				(font
+					(size 1.27 1.27)
+				)
+				(justify right)
+			)
+		)
+		(property "Footprint" "CellKeeper_Local:Capacitor_SMD__C_0805_2012Metric"
+			(at 391.16 299.72 0)
+			(hide yes)
+			(show_name no)
+			(do_not_autoplace no)
+			(effects
+				(font
+					(size 1.27 1.27)
+				)
+			)
+		)
+		(property "Datasheet" ""
+			(at 391.16 299.72 0)
+			(hide yes)
+			(show_name no)
+			(do_not_autoplace no)
+			(effects
+				(font
+					(size 1.27 1.27)
+				)
+			)
+		)
+		(property "Description" "10uF 50V X5R ±10% 0805 Multilayer Ceramic Capacitors MLCC - SMD/SMT ROHS"
+			(at 391.16 299.72 0)
+			(hide yes)
+			(show_name no)
+			(do_not_autoplace no)
+			(effects
+				(font
+					(size 1.27 1.27)
+				)
+			)
+		)
+		(property "JLCPCB Part #" "C440198"
+			(at 391.16 299.72 0)
+			(hide yes)
+			(show_name no)
+			(do_not_autoplace no)
+			(effects
+				(font
+					(size 1.27 1.27)
+				)
+			)
+		)
+		(property "Voltage" "50V X5R"
+			(at 386.842 302.514 0)
+			(show_name no)
+			(do_not_autoplace no)
+			(effects
+				(font
+					(size 1.27 1.27)
+				)
+				(justify right)
+			)
+		)
+		(pin "1"
+		)
+		(pin "2"
+		)
+		(instances
+			(project "CellKeeper"
+				(path "/5d962221-5e0a-481f-afc5-67c7ec101fc1"
+					(reference "C116")
+					(unit 1)
+				)
+			)
+		)
+	)
+	(symbol
 		(lib_id "CellKeeper_Local:power__GND")
 		(at 702.31 78.74 0)
@@
 	)
 	(symbol
-		(lib_id "CellKeeper_Local:Device__C_Small")
-		(at 391.16 299.72 180)
-		(unit 1)
-		(body_style 1)
-		(exclude_from_sim no)
-		(in_bom yes)
-		(on_board yes)
-		(in_pos_files yes)
-		(dnp no)
-		(property "Reference" "C57"
-			(at 385.318 299.72 0)
-			(show_name no)
-			(do_not_autoplace no)
-			(effects
-				(font
-					(size 1.27 1.27)
-				)
-				(justify right)
-			)
-		)
-		(property "Value" "1uF"
-			(at 385.572 301.752 0)
-			(show_name no)
-			(do_not_autoplace no)
-			(effects
-				(font
-					(size 1.27 1.27)
-				)
-				(justify right)
-			)
-		)
-		(property "Footprint" "CellKeeper_Local:Capacitor_SMD__C_0603_1608Metric"
-			(at 391.16 299.72 0)
-			(hide yes)
-			(show_name no)
-			(do_not_autoplace no)
-			(effects
-				(font
-					(size 1.27 1.27)
-				)
-			)
-		)
-		(property "Datasheet" ""
-			(at 391.16 299.72 0)
-			(hide yes)
-			(show_name no)
-			(do_not_autoplace no)
-			(effects
-				(font
-					(size 1.27 1.27)
-				)
-			)
-		)
-		(property "Description" "CL10A105KB8NNNC - 1uF 50V X5R ±10%"
-			(at 391.16 299.72 0)
-			(hide yes)
-			(show_name no)
-			(do_not_autoplace no)
-			(effects
-				(font
-					(size 1.27 1.27)
-				)
-			)
-		)
-		(property "JLCPCB Part #" "C15849"
-			(at 391.16 299.72 0)
-			(hide yes)
-			(show_name no)
-			(do_not_autoplace no)
-			(effects
-				(font
-					(size 1.27 1.27)
-				)
-			)
-		)
-		(pin "1"
-		)
-		(pin "2"
-		)
-		(instances
-			(project "CellKeeper"
-				(path "/5d962221-5e0a-481f-afc5-67c7ec101fc1"
-					(reference "C57")
-					(unit 1)
-				)
-			)
-		)
-	)
-	(symbol
 		(lib_id "CellKeeper_Local:BMS_Library__Jumper_Resistor")
 		(at 191.77 317.5 0)
@@
 		)
 		(property "Voltage" "50V X5R"
-			(at 333.248 305.054 0)
+			(at 328.422 305.562 0)
 			(show_name no)
 			(do_not_autoplace no)
